File: Hardware/NFC_Toy_KiCAD/NFC_Toy.sch (KiCad schematic (older format))
At the start: 50 parts, among them J1 Pad, J2 Pad, J3 JLink_Mini, U1 TPS61032, U19 MIC5225, U2 STM32L0-LQFP48, U3 LIS3DH

Commit message: Submitted to PCBWay for build
Parts:
- removed TP11, TP16, TP17, TP5: TEST, NFC_Toy_Lib:Test_Point, symbol TEST
Changed lines of the file:
@@
 	8380 3530 8180 3530
 Wire Wire Line
-	8180 3430 8180 3580
+	8180 3430 8180 3530
+Wire Wire Line
+	8180 3530 8180 3580
 Wire Wire Line
 	8380 3430 8180 3430
@@
 	2070 4630 2070 4730
 Wire Wire Line
-	1360 1730 2010 1730
+	1360 1730 1460 1730
+Wire Wire Line
+	1460 1730 1660 1730
+Wire Wire Line
+	1660 1730 2010 1730
 Wire Wire Line
 	1460 1730 1460 1780
@@
 	1460 1380 1360 1380
 Wire Wire Line
-	1460 1180 1460 1380
+	1460 1180 1460 1230
+Wire Wire Line
+	1460 1230 1460 1380
 Wire Wire Line
 	1660 1280 1660 1230
 Wire Wire Line
-	1460 1230 2710 1230
+	1460 1230 1660 1230
+Wire Wire Line
+	1660 1230 2010 1230
+Wire Wire Line
+	2010 1230 2210 1230
+Wire Wire Line
+	2210 1230 2360 1230
+Wire Wire Line
+	2360 1230 2610 1230
+Wire Wire Line
+	2610 1230 2710 1230
 Wire Wire Line
 	2010 1230 2010 1280
@@
 Connection ~ 2210 1230
 Wire Wire Line
-	2210 2030 2710 2030
+	2210 2030 2650 2030
+Wire Wire Line
+	2650 2030 2710 2030
 Wire Wire Line
 	2710 2130 2650 2130
@@
 	2210 2030 2210 1980
 Wire Wire Line
-	2360 1680 2360 2180
+	2360 1680 2360 1730
+Wire Wire Line
+	2360 1730 2360 2180
 Wire Wire Line
 	2360 1730 2710 1730
@@
 Connection ~ 1460 1230
 Wire Wire Line
-	4110 1630 5410 1630
-Wire Wire Line
-	4310 1430 4310 1680
+	4110 1630 4310 1630
+Wire Wire Line
+	4310 1630 4710 1630
+Wire Wire Line
+	4710 1630 5060 1630
+Wire Wire Line
+	5060 1630 5310 1630
+Wire Wire Line
+	5310 1630 5410 1630
+Wire Wire Line
+	4310 1430 4310 1530
+Wire Wire Line
+	4310 1530 4310 1630
+Wire Wire Line
+	4310 1630 4310 1680
 Wire Wire Line
 	4110 1530 4310 1530
@@
 Connection ~ 4310 1530
 Wire Wire Line
-	4710 1530 4710 1680
+	4710 1530 4710 1630
+Wire Wire Line
+	4710 1630 4710 1680
 Wire Wire Line
 	4310 2030 4310 1980
@@
 	6610 1730 6810 1730
 Wire Wire Line
-	6810 1680 6810 1780
+	6810 1680 6810 1730
+Wire Wire Line
+	6810 1730 6810 1780
 Wire Wire Line
 	6810 2080 6810 2180
@@
 	2560 4430 2660 4430
 Wire Wire Line
-	2560 4080 2560 4630
+	2560 4080 2560 4130
+Wire Wire Line
+	2560 4130 2560 4230
+Wire Wire Line
+	2560 4230 2560 4330
+Wire Wire Line
+	2560 4330 2560 4430
+Wire Wire Line
+	2560 4430 2560 4630
 Wire Wire Line
 	2660 4130 2560 4130
@@
 	2660 6830 2510 6830
 Wire Wire Line
-	2510 6830 2510 7180
+	2510 6830 2510 6930
+Wire Wire Line
+	2510 6930 2510 7030
+Wire Wire Line
+	2510 7030 2510 7130
+Wire Wire Line
+	2510 7130 2510 7180
 Wire Wire Line
 	2660 6930 2510 6930
@@
 	5860 5830 5960 5830
 Wire Wire Line
-	5860 4830 7060 4830
-Wire Wire Line
-	5860 4730 7060 4730
-Wire Wire Line
-	5860 5330 6550 5330
-Wire Wire Line
-	5860 5430 6550 5430
+	5860 4830 6940 4830
+Wire Wire Line
+	6940 4830 7060 4830
+Wire Wire Line
+	5860 4730 6570 4730
+Wire Wire Line
+	6570 4730 6710 4730
+Wire Wire Line
+	6710 4730 7060 4730
+Wire Wire Line
+	5860 5330 6250 5330
+Wire Wire Line
+	6250 5330 6550 5330
+Wire Wire Line
+	5860 5430 6470 5430
+Wire Wire Line
+	6470 5430 6550 5430
 Wire Wire Line
 	5960 5530 5860 5530
 Wire Wire Line
-	5860 5630 6760 5630
-Wire Wire Line
-	1460 5330 2660 5330
-Wire Wire Line
-	1460 5430 2660 5430
-Wire Wire Line
-	1460 5530 2660 5530
-Wire Wire Line
-	1460 5630 2660 5630
+	5860 5630 6700 5630
+Wire Wire Line
+	6700 5630 6760 5630
+Wire Wire Line
+	1460 5330 2040 5330
+Wire Wire Line
+	2040 5330 2660 5330
+Wire Wire Line
+	1460 5430 1860 5430
+Wire Wire Line
+	1860 5430 2660 5430
+Wire Wire Line
+	1460 5530 1680 5530
+Wire Wire Line
+	1680 5530 2660 5530
+Wire Wire Line
+	1460 5630 1500 5630
+Wire Wire Line
+	1500 5630 2660 5630
 Wire Wire Line
 	6710 4330 6710 4230
 Wire Wire Line
-	6710 4230 6940 4230
+	6710 4230 6810 4230
+Wire Wire Line
+	6810 4230 6940 4230
 Wire Wire Line
 	6940 4230 6940 4330
 Connection ~ 6810 4230
 Wire Wire Line
-	1760 4090 1760 4190
-Wire Wire Line
-	1760 4490 1760 4590
+	1760 4090 1760 4140
+Wire Wire Line
+	1760 4140 1760 4190
+Wire Wire Line
+	1760 4490 1760 4540
+Wire Wire Line
+	1760 4540 1760 4590
 Wire Wire Line
 	760  4490 760  4540
 Wire Wire Line
-	760  4540 1760 4540
+	760  4540 1010 4540
+Wire Wire Line
+	1010 4540 1260 4540
+Wire Wire Line
+	1260 4540 1510 4540
+Wire Wire Line
+	1510 4540 1760 4540
 Connection ~ 1760 4540
 Wire Wire Line
 	760  4190 760  4140
 Wire Wire Line
-	760  4140 1760 4140
+	760  4140 1010 4140
+Wire Wire Line
+	1010 4140 1260 4140
+Wire Wire Line
+	1260 4140 1510 4140
+Wire Wire Line
+	1510 4140 1760 4140
 Connection ~ 1760 4140
 Wire Wire Line
@@
 Connection ~ 1510 4540
 Wire Wire Line
-	8390 4950 8390 5150
+	8390 4950 8390 5000
+Wire Wire Line
+	8390 5000 8390 5050
+Wire Wire Line
+	8390 5050 8390 5150
 Wire Wire Line
 	8390 5150 8490 5150
@@
 	8390 5550 8490 5550
 Wire Wire Line
-	8390 5250 8390 5950
+	8390 5250 8390 5450
+Wire Wire Line
+	8390 5450 8390 5550
+Wire Wire Line
+	8390 5550 8390 5650
+Wire Wire Line
+	8390 5650 8390 5750
+Wire Wire Line
+	8390 5750 8390 5850
+Wire Wire Line
+	8390 5850 8390 5950
 Wire Wire Line
 	8490 5650 8390 5650
@@
 	8090 5050 8090 5000
 Wire Wire Line
-	7840 5000 8390 5000
+	7840 5000 8090 5000
+Wire Wire Line
+	8090 5000 8390 5000
 Connection ~ 8390 5000
 Wire Wire Line
@@
 	7470 3640 660  3640
 Wire Wire Line
-	6940 4630 6940 4980
+	6940 4630 6940 4830
+Wire Wire Line
+	6940 4830 6940 4980
 Connection ~ 6940 4830
 $Comp
@@
 	1680 5670 1680 5530
 Connection ~ 1680 5530
-$Comp
-L TEST TP5
-U 1 1 5AD39F6E
-P 7970 910
-F 0 "TP5" H 7970 1210 50  0000 C BNN
-F 1 "TEST" H 7970 1160 50  0000 C CNN
-F 2 "NFC_Toy_Lib:Test_Point" H 7970 910 50  0001 C CNN
-F 3 "" H 7970 910 50  0001 C CNN
-	1    7970 910
-	1    0    0    -1
-$EndComp
 NoConn ~ 5860 4330
 NoConn ~ 5860 6030
@@
 $EndComp
 Wire Wire Line
-	8330 1000 8330 850
+	8330 1000 8330 970
+Wire Wire Line
+	8330 970  8330 850
 Wire Wire Line
 	2660 5130 2620 5130
@@
 Connection ~ 1500 5630
 Wire Wire Line
-	2560 2530 2560 3080
-$Comp
-L TEST TP17
-U 1 1 5AE3537D
-P 7770 900
-F 0 "TP17" H 7770 1200 50  0000 C BNN
-F 1 "TEST" H 7770 1150 50  0000 C CNN
-F 2 "NFC_Toy_Lib:Test_Point" H 7770 900 50  0001 C CNN
-F 3 "" H 7770 900 50  0001 C CNN
-	1    7770 900
-	1    0    0    -1
-$EndComp
-$Comp
-L TEST TP16
-U 1 1 5AE3544B
-P 7570 900
-F 0 "TP16" H 7570 1200 50  0000 C BNN
-F 1 "TEST" H 7570 1150 50  0000 C CNN
-F 2 "NFC_Toy_Lib:Test_Point" H 7570 900 50  0001 C CNN
-F 3 "" H 7570 900 50  0001 C CNN
-	1    7570 900
-	1    0    0    -1
-$EndComp
-$Comp
-L TEST TP11
-U 1 1 5AE35510
-P 7380 900
-F 0 "TP11" H 7380 1200 50  0000 C BNN
-F 1 "TEST" H 7380 1150 50  0000 C CNN
-F 2 "NFC_Toy_Lib:Test_Point" H 7380 900 50  0001 C CNN
-F 3 "" H 7380 900 50  0001 C CNN
-	1    7380 900
-	1    0    0    -1
-$EndComp
-Wire Wire Line
-	7380 900  7380 970
-Wire Wire Line
-	7380 970  8330 970
-Connection ~ 8330 970
-Wire Wire Line
-	7970 910  7970 970
-Connection ~ 7970 970
-Wire Wire Line
-	7770 900  7770 970
-Connection ~ 7770 970
-Wire Wire Line
-	7570 900  7570 970
-Connection ~ 7570 970
+	2560 2530 2560 2630
+Wire Wire Line
+	2560 2630 2560 2730
+Wire Wire Line
+	2560 2730 2560 2830
+Wire Wire Line
+	2560 2830 2560 3030
+Wire Wire Line
+	2560 3030 2560 3080
 Wire Wire Line
 	2710 2530 2560 2530

Commit message: Added RNG and "Try Again"
Parts:
- C1, C10, C11, C12, C13, C2, C3, C4, C5, C6, C7, C8: symbol C -> Device:C
- C9: symbol CP1 -> Device:CP1
- D1, D2: symbol LED -> Device:LED
- J1, J2: symbol Pad -> Pad:Pad
- J3: symbol JLink_Mini -> JLink_Mini:JLink_Mini
- L1: symbol L -> Device:L
- MK1, MK2, MK3, MK4: symbol Mounting_Hole -> NFC_Toy-rescue:Mounting_Hole
- R1, R10, R2, R3, R4, R5, R6, R7, R8, R9: symbol R -> Device:R
- TP1, TP10, TP2, TP3, TP4, TP6, TP7, TP8, TP9: symbol TEST -> NFC_Toy-rescue:TEST
- U1: symbol TPS61030 -> TPS61030:TPS61030
- U19: symbol MIC5225 -> MIC5225:MIC5225
- U2: symbol STM32L0-LQFP48 -> STM32L0-LQFP48:STM32L0-LQFP48
- U3: symbol LIS3DH -> LIS3DH:LIS3DH
