File: Hardware/NFC_Toy_KiCAD/NFC_Toy_Audio.sch (KiCad schematic (older format))
At the start: 6 parts

Commit message: Ready to start layout
Parts:
- added C14, C15: 0.1u, symbol C
- added C16: 10u, symbol C
- gave numbers to parts that had none: 6
Connections:
- net +3V3: now also C14.1
- net +5V: now also C15.1, C16.1
- net GND: now also C14.2, C15.2, C16.2
Other:
- moved on the sheet: J15, J16, J17, R11, R12, U4

Commit message: Layout started
Parts:
- C14, C15: footprint (none) -> Capacitors_SMD:C_0402
- C16: footprint (none) -> Capacitors_SMD:C_0603_HandSoldering
- J4: renamed from J16; footprint (none) -> NFC_Toy_Lib:Pad_SMD_Small
- J5: renamed from J17; footprint (none) -> NFC_Toy_Lib:Pad_SMD_Small
- J6: renamed from J15; footprint MOLEX_503182-1852 -> NFC_Toy_Lib:MOLEX_503182-1852
- R11, R12: footprint (none) -> Resistors_SMD:R_0603_HandSoldering
- U4: footprint MODULE -> NFC_Toy_Lib:QFN50P300X300X80-17N
Connections:
- net GND: now also U4.17 (PWRPAD)
Changed lines of the file:
@@
 F 0 "U4" H 7040 3530 50  0000 C CNN
 F 1 "MAX98357" H 7040 3730 50  0000 C CNN
-F 2 "MODULE" H 7040 3630 50  0001 C CNN
+F 2 "NFC_Toy_Lib:QFN50P300X300X80-17N" H 7040 3630 50  0001 C CNN
 F 3 "DOCUMENTATION" H 7040 3630 50  0001 C CNN
 	1    7040 3630
@@
 NoConn ~ 6140 3830
 $Comp
-L GND #PWR39
+L GND #PWR038
 U 1 1 5ACDFE68
 P 7040 4580
-F 0 "#PWR39" H 7040 4330 50  0001 C CNN
+F 0 "#PWR038" H 7040 4330 50  0001 C CNN
 F 1 "GND" H 7040 4430 50  0000 C CNN
 F 2 "" H 7040 4580 50  0001 C CNN
@@
 $EndComp
 $Comp
-L +5V #PWR40
+L +5V #PWR039
 U 1 1 5ACDFE6E
 P 7090 2380
-F 0 "#PWR40" H 7090 2230 50  0001 C CNN
+F 0 "#PWR039" H 7090 2230 50  0001 C CNN
 F 1 "+5V" H 7090 2520 50  0000 C CNN
 F 2 "" H 7090 2380 50  0001 C CNN
@@
 	6940 4530 6940 4580
 Wire Wire Line
-	6940 4580 7140 4580
+	6940 4580 7290 4580
 Wire Wire Line
 	7140 4580 7140 4530
@@
 F 0 "R11" V 5470 3230 50  0000 C CNN
 F 1 "DNP" V 5390 3230 50  0000 C CNN
-F 2 "" V 5320 3230 50  0001 C CNN
+F 2 "Resistors_SMD:R_0603_HandSoldering" V 5320 3230 50  0001 C CNN
 F 3 "" H 5390 3230 50  0001 C CNN
 	1    5390 3230
@@
 F 0 "R12" V 5470 3630 50  0000 C CNN
 F 1 "DNP" V 5390 3630 50  0000 C CNN
-F 2 "" V 5320 3630 50  0001 C CNN
+F 2 "Resistors_SMD:R_0603_HandSoldering" V 5320 3630 50  0001 C CNN
 F 3 "" H 5390 3630 50  0001 C CNN
 	1    5390 3630
@@
 Connection ~ 5390 3430
 $Comp
-L GND #PWR38
+L GND #PWR040
 U 1 1 5ACDFE90
 P 5390 3830
-F 0 "#PWR38" H 5390 3580 50  0001 C CNN
+F 0 "#PWR040" H 5390 3580 50  0001 C CNN
 F 1 "GND" H 5390 3680 50  0000 C CNN
 F 2 "" H 5390 3830 50  0001 C CNN
@@
 $EndComp
 $Comp
-L +5V #PWR37
+L +5V #PWR041
 U 1 1 5ACDFE96
 P 5390 3030
-F 0 "#PWR37" H 5390 2880 50  0001 C CNN
+F 0 "#PWR041" H 5390 2880 50  0001 C CNN
 F 1 "+5V" H 5390 3170 50  0000 C CNN
 F 2 "" H 5390 3030 50  0001 C CNN
@@
 GAIN_SLOT:\n    100k to GND - 15dB\n    GND - 12dB\n    NC - 9dB\n    VDD - 6dB\n    100k to VDD - 3dB
 $Comp
-L Pad J16
+L Pad J4
 U 1 1 5ACE08A3
 P 8540 3730
-F 0 "J16" H 8540 3530 60  0000 C CNN
+F 0 "J4" H 8540 3530 60  0000 C CNN
 F 1 "SPKR-" H 8540 3730 60  0000 C CNN
-F 2 "" H 8540 3730 60  0001 C CNN
+F 2 "NFC_Toy_Lib:Pad_SMD_Small" H 8540 3730 60  0001 C CNN
 F 3 "" H 8540 3730 60  0001 C CNN
 	1    8540 3730
@@
 $EndComp
 $Comp
-L Pad J17
+L Pad J5
 U 1 1 5ACE08AA
 P 8540 4080
-F 0 "J17" H 8540 3880 60  0000 C CNN
+F 0 "J5" H 8540 3880 60  0000 C CNN
 F 1 "SPKR+" H 8540 4080 60  0000 C CNN
-F 2 "" H 8540 4080 60  0001 C CNN
+F 2 "NFC_Toy_Lib:Pad_SMD_Small" H 8540 4080 60  0001 C CNN
 F 3 "" H 8540 4080 60  0001 C CNN
 	1    8540 4080
@@
 $EndComp
 $Comp
-L 503182-1852 J15
+L 503182-1852 J6
 U 1 1 5ACE08EE
 P 3240 3580
-F 0 "J15" H 3240 4303 50  0000 L BNN
+F 0 "J6" H 3240 4303 50  0000 L BNN
 F 1 "503182-1852" H 3240 2757 50  0000 L BNN
-F 2 "MOLEX_503182-1852" H 3240 3580 50  0001 L BNN
+F 2 "NFC_Toy_Lib:MOLEX_503182-1852" H 3240 3580 50  0001 L BNN
 F 3 "5031821852" H 3240 3580 50  0001 L BNN
 F 4 "Unavailable" H 3240 3580 50  0001 L BNN "Field4"
@@
 	3690 3080 3440 3080
 $Comp
-L +3.3V #PWR34
+L +3.3V #PWR042
 U 1 1 5ACE0C10
 P 3590 2450
-F 0 "#PWR34" H 3590 2300 50  0001 C CNN
+F 0 "#PWR042" H 3590 2300 50  0001 C CNN
 F 1 "+3.3V" H 3590 2590 50  0000 C CNN
 F 2 "" H 3590 2450 50  0001 C CNN
@@
 	3440 3980 3690 3980
 $Comp
-L GND #PWR35
+L GND #PWR043
 U 1 1 5ACE0D8F
 P 3590 4230
-F 0 "#PWR35" H 3590 3980 50  0001 C CNN
+F 0 "#PWR043" H 3590 3980 50  0001 C CNN
 F 1 "GND" H 3590 4080 50  0000 C CNN
 F 2 "" H 3590 4230 50  0001 C CNN
@@
 F 0 "C14" H 3805 2740 50  0000 L CNN
 F 1 "0.1u" H 3805 2540 50  0000 L CNN
-F 2 "" H 3818 2490 50  0001 C CNN
+F 2 "Capacitors_SMD:C_0402" H 3818 2490 50  0001 C CNN
 F 3 "" H 3780 2640 50  0001 C CNN
 	1    3780 2640
@@
 $EndComp
 $Comp
-L GND #PWR36
+L GND #PWR044
 U 1 1 5AD11F0E
 P 3780 2830
-F 0 "#PWR36" H 3780 2580 50  0001 C CNN
+F 0 "#PWR044" H 3780 2580 50  0001 C CNN
 F 1 "GND" H 3780 2680 50  0000 C CNN
 F 2 "" H 3780 2830 50  0001 C CNN
@@
 F 0 "C15" H 7395 2670 50  0000 L CNN
 F 1 "0.1u" H 7395 2470 50  0000 L CNN
-F 2 "" H 7408 2420 50  0001 C CNN
+F 2 "Capacitors_SMD:C_0402" H 7408 2420 50  0001 C CNN
 F 3 "" H 7370 2570 50  0001 C CNN
 	1    7370 2570
@@
 $EndComp
 $Comp
-L GND #PWR41
+L GND #PWR045
 U 1 1 5AD12414
 P 7370 2750
-F 0 "#PWR41" H 7370 2500 50  0001 C CNN
+F 0 "#PWR045" H 7370 2500 50  0001 C CNN
 F 1 "GND" H 7370 2600 50  0000 C CNN
 F 2 "" H 7370 2750 50  0001 C CNN
@@
 F 0 "C16" H 7725 2670 50  0000 L CNN
 F 1 "10u" H 7725 2470 50  0000 L CNN
-F 2 "" H 7738 2420 50  0001 C CNN
+F 2 "Capacitors_SMD:C_0603_HandSoldering" H 7738 2420 50  0001 C CNN
 F 3 "" H 7700 2570 50  0001 C CNN
 	1    7700 2570
@@
 $EndComp
 $Comp
-L GND #PWR42
+L GND #PWR046
 U 1 1 5AD125D7
 P 7700 2760
-F 0 "#PWR42" H 7700 2510 50  0001 C CNN
+F 0 "#PWR046" H 7700 2510 50  0001 C CNN
 F 1 "GND" H 7700 2610 50  0000 C CNN
 F 2 "" H 7700 2760 50  0001 C CNN
@@
 	7700 2380 7700 2420
 Connection ~ 7370 2380
+Connection ~ 7140 4580
+Wire Wire Line
+	7290 4580 7290 4530
 $EndSCHEMATC

Commit message: Added RNG and "Try Again"
Parts:
- C?: renamed from C14; symbol C -> Device:C
- C?: renamed from C15; symbol C -> Device:C
- C?: renamed from C16; symbol C -> Device:C
- J?: renamed from J4; symbol Pad -> Pad:Pad
- J?: renamed from J5; symbol Pad -> Pad:Pad
- J?: renamed from J6; symbol 503182-1852 -> Micro-SD-503182-1852:503182-1852
- R?: renamed from R11; symbol R -> Device:R
- R?: renamed from R12; symbol R -> Device:R
- U?: renamed from U4; symbol MAX98357 -> MAX98357:MAX98357
Changed lines of the file:
@@
-EESchema Schematic File Version 2
-LIBS:power
-LIBS:device
-LIBS:transistors
-LIBS:conn
-LIBS:linear
-LIBS:regul
-LIBS:74xx
-LIBS:cmos4000
-LIBS:adc-dac
-LIBS:memory
-LIBS:xilinx
-LIBS:microcontrollers
-LIBS:dsp
-LIBS:microchip
-LIBS:analog_switches
-LIBS:motorola
-LIBS:texas
-LIBS:intel
-LIBS:audio
-LIBS:interface
-LIBS:digital-audio
-LIBS:philips
-LIBS:display
-LIBS:cypress
-LIBS:siliconi
-LIBS:opto
-LIBS:atmel
-LIBS:contrib
-LIBS:valves
-LIBS:stm32
-LIBS:JLink_Mini
-LIBS:STM32L062K8
-LIBS:Pad
-LIBS:LIS3DH
-LIBS:TPS61030
-LIBS:MIC5225
-LIBS:STM32L0-LQFP48
-LIBS:MAX98357
-LIBS:Micro SD 503182-1852
-LIBS:PN532
-LIBS:Oscillator
-LIBS:APA102
-LIBS:SN74LVC2T45
-LIBS:mechanical
+EESchema Schematic File Version 4
+LIBS:CommandCenter_KICAD-cache
 LIBS:NFC_Toy-cache
-EELAYER 25 0
+EELAYER 29 0
 EELAYER END
 $Descr A4 11693 8268
@@
 $EndDescr
 $Comp
-L MAX98357 U4
+L MAX98357:MAX98357 U?
 U 1 1 5ACDFE57
 P 7040 3630
-F 0 "U4" H 7040 3530 50  0000 C CNN
+F 0 "U?" H 7040 3530 50  0000 C CNN
 F 1 "MAX98357" H 7040 3730 50  0000 C CNN
 F 2 "NFC_Toy_Lib:QFN50P300X300X80-17N" H 7040 3630 50  0001 C CNN
@@
 NoConn ~ 6140 3830
 $Comp
-L GND #PWR034
+L power:GND #PWR?
 U 1 1 5ACDFE68
 P 7040 4580
-F 0 "#PWR034" H 7040 4330 50  0001 C CNN
+F 0 "#PWR?" H 7040 4330 50  0001 C CNN
 F 1 "GND" H 7040 4430 50  0000 C CNN
 F 2 "" H 7040 4580 50  0001 C CNN
@@
 $EndComp
 $Comp
-L +5V #PWR035
+L power:+5V #PWR?
 U 1 1 5ACDFE6E
 P 7090 2380
-F 0 "#PWR035" H 7090 2230 50  0001 C CNN
+F 0 "#PWR?" H 7090 2230 50  0001 C CNN
 F 1 "+5V" H 7090 2520 50  0000 C CNN
 F 2 "" H 7090 2380 50  0001 C CNN
@@
 	6040 3330 6140 3330
 $Comp
-L R R11
+L Device:R R?
 U 1 1 5ACDFE7F
 P 5390 3230
-F 0 "R11" V 5470 3230 50  0000 C CNN
+F 0 "R?" V 5470 3230 50  0000 C CNN
 F 1 "DNP" V 5390 3230 50  0000 C CNN
 F 2 "Resistors_SMD:R_0603_HandSoldering" V 5320 3230 50  0001 C CNN
@@
 $EndComp
 $Comp
-L R R12
+L Device:R R?
 U 1 1 5ACDFE86
 P 5390 3630
-F 0 "R12" V 5470 3630 50  0000 C CNN
+F 0 "R?" V 5470 3630 50  0000 C CNN
 F 1 "DNP" V 5390 3630 50  0000 C CNN
 F 2 "Resistors_SMD:R_0603_HandSoldering" V 5320 3630 50  0001 C CNN
@@
 Connection ~ 5390 3430
 $Comp
-L GND #PWR036
+L power:GND #PWR?
 U 1 1 5ACDFE90
 P 5390 3830
-F 0 "#PWR036" H 5390 3580 50  0001 C CNN
+F 0 "#PWR?" H 5390 3580 50  0001 C CNN
 F 1 "GND" H 5390 3680 50  0000 C CNN
 F 2 "" H 5390 3830 50  0001 C CNN
@@
 $EndComp
 $Comp
-L +5V #PWR037
+L power:+5V #PWR?
 U 1 1 5ACDFE96
 P 5390 3030
-F 0 "#PWR037" H 5390 2880 50  0001 C CNN
+F 0 "#PWR?" H 5390 2880 50  0001 C CNN
 F 1 "+5V" H 5390 3170 50  0000 C CNN
 F 2 "" H 5390 3030 50  0001 C CNN
@@
 GAIN_SLOT:\n    100k to GND - 15dB\n    GND - 12dB\n    NC - 9dB\n    VDD - 6dB\n    100k to VDD - 3dB
 $Comp
-L Pad J4
+L Pad:Pad J?
 U 1 1 5ACE08A3
 P 8540 3730
-F 0 "J4" H 8540 3530 60  0000 C CNN
+F 0 "J?" H 8540 3530 60  0000 C CNN
 F 1 "SPKR-" H 8540 3730 60  0000 C CNN
 F 2 "NFC_Toy_Lib:Pad_SMD_Small" H 8540 3730 60  0001 C CNN
@@
 $EndComp
 $Comp
-L Pad J5
+L Pad:Pad J?
 U 1 1 5ACE08AA
 P 8540 4080
-F 0 "J5" H 8540 3880 60  0000 C CNN
+F 0 "J?" H 8540 3880 60  0000 C CNN
 F 1 "SPKR+" H 8540 4080 60  0000 C CNN
 F 2 "NFC_Toy_Lib:Pad_SMD_Small" H 8540 4080 60  0001 C CNN
@@
 $EndComp
 $Comp
-L 503182-1852 J6
+L Micro-SD-503182-1852:503182-1852 J?
 U 1 1 5ACE08EE
 P 3240 3580
-F 0 "J6" H 3240 4303 50  0000 L BNN
+F 0 "J?" H 3240 4303 50  0000 L BNN
 F 1 "503182-1852" H 3240 2757 50  0000 L BNN
 F 2 "NFC_Toy_Lib:MOLEX_503182-1852" H 3240 3580 50  0001 L BNN
@@
 	3690 3080 3440 3080
 $Comp
-L +3.3V #PWR038
+L power:+3.3V #PWR?
 U 1 1 5ACE0C10
 P 3590 2450
-F 0 "#PWR038" H 3590 2300 50  0001 C CNN
+F 0 "#PWR?" H 3590 2300 50  0001 C CNN
 F 1 "+3.3V" H 3590 2590 50  0000 C CNN
 F 2 "" H 3590 2450 50  0001 C CNN
@@
 	3440 3980 3690 3980
 $Comp
-L GND #PWR039
+L power:GND #PWR?
 U 1 1 5ACE0D8F
 P 3590 4230
-F 0 "#PWR039" H 3590 3980 50  0001 C CNN
+F 0 "#PWR?" H 3590 3980 50  0001 C CNN
 F 1 "GND" H 3590 4080 50  0000 C CNN
 F 2 "" H 3590 4230 50  0001 C CNN
@@
 	8090 4180 8290 4180
 $Comp
-L C C14
+L Device:C C?
 U 1 1 5AD11D71
 P 3780 2640
-F 0 "C14" H 3805 2740 50  0000 L CNN
+F 0 "C?" H 3805 2740 50  0000 L CNN
 F 1 "0.1u" H 3805 2540 50  0000 L CNN
 F 2 "Capacitors_SMD:C_0402" H 3818 2490 50  0001 C CNN
@@
 $EndComp
 $Comp
-L GND #PWR040
+L power:GND #PWR?
 U 1 1 5AD11F0E
 P 3780 2830
-F 0 "#PWR040" H 3780 2580 50  0001 C CNN
+F 0 "#PWR?" H 3780 2580 50  0001 C CNN
 F 1 "GND" H 3780 2680 50  0000 C CNN
 F 2 "" H 3780 2830 50  0001 C CNN
@@
 	3780 2790 3780 2830
 $Comp
-L C C15
+L Device:C C?
 U 1 1 5AD1240E
 P 7370 2570
-F 0 "C15" H 7395 2670 50  0000 L CNN
+F 0 "C?" H 7395 2670 50  0000 L CNN
 F 1 "0.1u" H 7395 2470 50  0000 L CNN
 F 2 "Capacitors_SMD:C_0402" H 7408 2420 50  0001 C CNN
@@
 $EndComp
 $Comp
-L GND #PWR041
+L power:GND #PWR?
 U 1 1 5AD12414
 P 7370 2750
-F 0 "#PWR041" H 7370 2500 50  0001 C CNN
+F 0 "#PWR?" H 7370 2500 50  0001 C CNN
 F 1 "GND" H 7370 2600 50  0000 C CNN
 F 2 "" H 7370 2750 50  0001 C CNN
@@
 	7370 2720 7370 2750
 $Comp
-L C C16
+L Device:C C?
 U 1 1 5AD12566
 P 7700 2570
-F 0 "C16" H 7725 2670 50  0000 L CNN
+F 0 "C?" H 7725 2670 50  0000 L CNN
 F 1 "10u" H 7725 2470 50  0000 L CNN
 F 2 "Capacitors_SMD:C_0603_HandSoldering" H 7738 2420 50  0001 C CNN
@@
 $EndComp
 $Comp
-L GND #PWR042
+L power:GND #PWR?
 U 1 1 5AD125D7
 P 7700 2760
-F 0 "#PWR042" H 7700 2510 50  0001 C CNN
+F 0 "#PWR?" H 7700 2510 50  0001 C CNN
 F 1 "GND" H 7700 2610 50  0000 C CNN
 F 2 "" H 7700 2760 50  0001 C CNN
